File: LS4.kicad_sch (KiCad schematic)
At the start: 0 parts

Commit message: colocacion de los componentes en un 90%
Parts:
- added R16, R37, R38, R39, R42, R43, R44, R45: 4.7k, hellen-one-common:R0603, symbol hellen-one-common:Res
- added U3, U9: VNLD5160TR-E, Package_SO:SOIC-8_3.9x4.9mm_P1.27mm, symbol chips:VNLD5160
Connections:
- new net: R44.2, U3.1 (IN1)
- new net: R45.2, U3.3 (IN2)
- new net: R43.2, U9.3 (IN2)
- new net: R42.2, U9.1 (IN1)
- new net GND: R16.2, R37.2, R38.2, R39.2, U3.5 (S2), U3.7 (S1), U9.5 (S2), U9.7 (S1)
- new net IN1: R16.1, R44.1
- new net IN2: R38.1, R45.1
- new net IN3: R37.1, R42.1
- new net IN4: R39.1, R43.1
- new net OUT1: U3.8 (D1)
- new net OUT2: U3.6 (D2)
- new net OUT3: U9.8 (D1)
- new net OUT4: U9.6 (D2)
- no-connect marks 0 -> 4
