File: egt.kicad_sch (KiCad schematic)
At the start: 9 parts, among them U6 MAX31855KASA

Commit message: colocacion de los componentes en un 90%
Parts:
- renumbered C29 to C28, C30 to C29, C31 to C30, C32 to C31, C33 to C32, U6 to U8
Changed lines of the file:
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@@
 		(on_board yes)
 		(dnp no)
-		(property "Reference" "U6"
+		(property "Reference" "U8"
 			(at 164.7541 80.01 0)
 			(effects
@@
 		(instances
 			(project "hellen121vag"
-				(path "/45c1f041-3b7c-4036-abe9-e26621c05a73/c375f9f4-5431-4085-b42f-ed4da13bcbaf"
-					(reference "U6")
+				(path "/45c1f041-3b7c-4036-abe9-e26621c05a73/6cde32b6-05f2-499d-9aff-ad44aab97055"
+					(reference "U8")
 					(unit 1)
 				)
@@
 		(instances
 			(project "hellen121vag"
-				(path "/45c1f041-3b7c-4036-abe9-e26621c05a73/c375f9f4-5431-4085-b42f-ed4da13bcbaf"
+				(path "/45c1f041-3b7c-4036-abe9-e26621c05a73/6cde32b6-05f2-499d-9aff-ad44aab97055"
 					(reference "L2")
 					(unit 1)
@@
 		(on_board yes)
 		(dnp no)
-		(property "Reference" "C32"
+		(property "Reference" "C31"
 			(at 175.26 71.755 90)
 			(effects
@@
 		(instances
 			(project "hellen121vag"
-				(path "/45c1f041-3b7c-4036-abe9-e26621c05a73/c375f9f4-5431-4085-b42f-ed4da13bcbaf"
-					(reference "C32")
+				(path "/45c1f041-3b7c-4036-abe9-e26621c05a73/6cde32b6-05f2-499d-9aff-ad44aab97055"
+					(reference "C31")
 					(unit 1)
 				)
@@
 		(on_board yes)
 		(dnp no)
-		(property "Reference" "#PWR0120"
+		(property "Reference" "#PWR0151"
 			(at 132.08 114.3 0)
 			(effects
@@
 		(instances
 			(project "hellen121vag"
-				(path "/45c1f041-3b7c-4036-abe9-e26621c05a73/c375f9f4-5431-4085-b42f-ed4da13bcbaf"
-					(reference "#PWR0120")
+				(path "/45c1f041-3b7c-4036-abe9-e26621c05a73/6cde32b6-05f2-499d-9aff-ad44aab97055"
+					(reference "#PWR0151")
 					(unit 1)
 				)
@@
 		(on_board yes)
 		(dnp no)
-		(property "Reference" "#PWR0123"
+		(property "Reference" "#PWR0154"
 			(at 172.72 83.82 0)
 			(effects
@@
 		(instances
 			(project "hellen121vag"
-				(path "/45c1f041-3b7c-4036-abe9-e26621c05a73/c375f9f4-5431-4085-b42f-ed4da13bcbaf"
-					(reference "#PWR0123")
+				(path "/45c1f041-3b7c-4036-abe9-e26621c05a73/6cde32b6-05f2-499d-9aff-ad44aab97055"
+					(reference "#PWR0154")
 					(unit 1)
 				)
@@
 		(on_board yes)
 		(dnp no)
-		(property "Reference" "C33"
+		(property "Reference" "C32"
 			(at 187.96 71.755 90)
 			(effects
@@
 		(instances
 			(project "hellen121vag"
-				(path "/45c1f041-3b7c-4036-abe9-e26621c05a73/c375f9f4-5431-4085-b42f-ed4da13bcbaf"
-					(reference "C33")
+				(path "/45c1f041-3b7c-4036-abe9-e26621c05a73/6cde32b6-05f2-499d-9aff-ad44aab97055"
+					(reference "C32")
 					(unit 1)
 				)
@@
 		(on_board yes)
 		(dnp no)
-		(property "Reference" "#PWR0122"
+		(property "Reference" "#PWR0155"
 			(at 162.56 111.76 0)
 			(effects
@@
 		(instances
 			(project "hellen121vag"
-				(path "/45c1f041-3b7c-4036-abe9-e26621c05a73/c375f9f4-5431-4085-b42f-ed4da13bcbaf"
-					(reference "#PWR0122")
+				(path "/45c1f041-3b7c-4036-abe9-e26621c05a73/6cde32b6-05f2-499d-9aff-ad44aab97055"
+					(reference "#PWR0155")
 					(unit 1)
 				)
@@
 		(on_board yes)
 		(dnp no)
-		(property "Reference" "C30"
+		(property "Reference" "C29"
 			(at 140.97 89.535 90)
 			(effects
@@
 		(instances
 			(project "hellen121vag"
-				(path "/45c1f041-3b7c-4036-abe9-e26621c05a73/c375f9f4-5431-4085-b42f-ed4da13bcbaf"
-					(reference "C30")
+				(path "/45c1f041-3b7c-4036-abe9-e26621c05a73/6cde32b6-05f2-499d-9aff-ad44aab97055"
+					(reference "C29")
 					(unit 1)
 				)
@@
 		(on_board yes)
 		(dnp no)
-		(property "Reference" "C29"
+		(property "Reference" "C28"
 			(at 134.62 99.695 90)
 			(effects
@@
 		(instances
 			(project "hellen121vag"
-				(path "/45c1f041-3b7c-4036-abe9-e26621c05a73/c375f9f4-5431-4085-b42f-ed4da13bcbaf"
-					(reference "C29")
+				(path "/45c1f041-3b7c-4036-abe9-e26621c05a73/6cde32b6-05f2-499d-9aff-ad44aab97055"
+					(reference "C28")
 					(unit 1)
 				)
@@
 		(on_board yes)
 		(dnp no)
-		(property "Reference" "#PWR0121"
+		(property "Reference" "#PWR0153"
 			(at 147.32 114.3 0)
 			(effects
@@
 		(instances
 			(project "hellen121vag"
-				(path "/45c1f041-3b7c-4036-abe9-e26621c05a73/c375f9f4-5431-4085-b42f-ed4da13bcbaf"
-					(reference "#PWR0121")
+				(path "/45c1f041-3b7c-4036-abe9-e26621c05a73/6cde32b6-05f2-499d-9aff-ad44aab97055"
+					(reference "#PWR0153")
 					(unit 1)
 				)
@@
 		(on_board yes)
 		(dnp no)
-		(property "Reference" "#PWR0124"
+		(property "Reference" "#PWR0156"
 			(at 185.42 83.82 0)
 			(effects
@@
 		(instances
 			(project "hellen121vag"
-				(path "/45c1f041-3b7c-4036-abe9-e26621c05a73/c375f9f4-5431-4085-b42f-ed4da13bcbaf"
-					(reference "#PWR0124")
+				(path "/45c1f041-3b7c-4036-abe9-e26621c05a73/6cde32b6-05f2-499d-9aff-ad44aab97055"
+					(reference "#PWR0156")
 					(unit 1)
 				)
@@
 		(instances
 			(project "hellen121vag"
-				(path "/45c1f041-3b7c-4036-abe9-e26621c05a73/c375f9f4-5431-4085-b42f-ed4da13bcbaf"
+				(path "/45c1f041-3b7c-4036-abe9-e26621c05a73/6cde32b6-05f2-499d-9aff-ad44aab97055"
 					(reference "D6")
 					(unit 1)
@@
 		(on_board yes)
 		(dnp no)
-		(property "Reference" "C31"
+		(property "Reference" "C30"
 			(at 149.86 99.695 90)
 			(effects
@@
 		(instances
 			(project "hellen121vag"
-				(path "/45c1f041-3b7c-4036-abe9-e26621c05a73/c375f9f4-5431-4085-b42f-ed4da13bcbaf"
-					(reference "C31")
+				(path "/45c1f041-3b7c-4036-abe9-e26621c05a73/6cde32b6-05f2-499d-9aff-ad44aab97055"
+					(reference "C30")
 					(unit 1)
 				)
@@
 		(instances
 			(project "hellen121vag"
-				(path "/45c1f041-3b7c-4036-abe9-e26621c05a73/c375f9f4-5431-4085-b42f-ed4da13bcbaf"
+				(path "/45c1f041-3b7c-4036-abe9-e26621c05a73/6cde32b6-05f2-499d-9aff-ad44aab97055"
 					(reference "L1")
 					(unit 1)
@@
 		(on_board yes)
 		(dnp no)
-		(property "Reference" "#PWR0119"
+		(property "Reference" "#PWR0152"
 			(at 115.57 114.3 0)
 			(effects
@@
 		(instances
 			(project "hellen121vag"
-				(path "/45c1f041-3b7c-4036-abe9-e26621c05a73/c375f9f4-5431-4085-b42f-ed4da13bcbaf"
-					(reference "#PWR0119")
-					(unit 1)
-				)
+				(path "/45c1f041-3b7c-4036-abe9-e26621c05a73/6cde32b6-05f2-499d-9aff-ad44aab97055"
+					(reference "#PWR0152")
+					(unit 1)
+				)
