File: hellen121vag.kicad_sch (KiCad schematic)
At the start: 111 parts, among them J1 USB_B_Mini, J10 AudioJack_THR, J2 Conn_01x01, J3 Conn_01x01, J4 Conn_01x01, J5 Conn_01x01, J6 Conn_01x01, J7 Conn_01x08, J8 Conn_01x06, M11 Module-vr-discrete-0.4, M3 mega-mcu144-0.1, M5 Module-knock-0.2, M6 Module-output-0.3, M7 Module-ign8-0.2, M8 Module-power_12and5V-0.1, M9 Module-wbo-0.5, P1 368255-2, P10 Pad, P11 Pad, P12 Pad, P13 Pad, P14 Pad, P15 Pad, P16 Pad, P17 Pad, P2 Pad, P20 Pad, P28 Pad, P3 Pad, P4 Pad, P40 Pad, P41 Pad, P43 Pad, P44 Pad, P45 Pad, P46 Pad, P48 Pad, P49 Pad, P5 Pad, P56 Pad, P6 Pad, P61 Pad, P63 Pad, P64 Pad, P66 Pad, P67 Pad, P68 Pad, P69 Pad, P7 Pad, P74 Pad, P8 Pad, P80 Pad, P9 Pad, U1 L6205PD, U3 MCP6002-xSN

Commit message: se modifico esquema y pcb
Parts:
- removed BT1: BATTERY_CR2032, Battery:BatteryHolder_Keystone_1060_1x2032, symbol art-electro-power:BATTERY_CR2032
- removed C10, C11, C12, C13, C14, C7, C8, C9: 10u, Capacitor_SMD:C_0805_2012Metric, symbol hellen-one-common:Cap
- removed C16, C2: 100n, hellen-one-common:C0603, symbol hellen-one-common:Cap
- removed C17: 10u, hellen-one-common:C0603, symbol hellen-one-common:Cap
- removed C3: 220n, hellen-one-common:C0603, symbol hellen-one-common:Cap
- removed C4: 10n, hellen-one-common:C0603, symbol hellen-one-common:Cap
- removed C5: 5.6n, hellen-one-common:C0603, symbol hellen-one-common:Cap
- removed D10, D11, D12, D13, D14: B5819W, Diode_SMD:D_SOD-123, symbol hellen-one-common:1N4148WS
- removed D4, D6, D7, D8: LED-GREEN-0805, hellen-one-common:LED-0805, symbol hellen-one-common:LED
- removed D9: 1N4148WS, hellen-one-common:SOD-323, symbol hellen-one-common:1N4148WS
- removed G3, G5: PROTO_AREA, hellen-one-common:PROTO_AREA, symbol hellen-one-common:PROTO_AREA
- removed G4: DISCLAIMER, rusefi_lib:Off_Road_Disclaimer, symbol Off_Road_Disclaimer:Disclaimer
- removed G6: LOGO, hellen-one-common:LOGO, symbol hellen-one-common:LOGO
- removed G7: LOGO, rusefi_lib:LOGO, symbol logo:LOGO
- removed J1: USB_B_Mini, hellen-one-common:USB-MINI-B-VERTICAL, symbol hellen-one-common:USB_B_Mini
- removed J10: AudioJack_THR, hellen-one-common:Jack_3.5mm_PJ-3250-5A, symbol hellen-one-common:AudioJack_THR
- removed J2, J3, J4, J5, J6: Conn_01x01, TestPoint:TestPoint_Pad_D2.0mm, symbol Connector_Generic:Conn_01x01
- removed J7: Conn_01x08, Connector_PinHeader_2.54mm:PinHeader_1x08_P2.54mm_Vertical, symbol Connector_Generic:Conn_01x08
- removed J8: Conn_01x06, Connector_PinHeader_2.54mm:PinHeader_1x06_P2.54mm_Vertical, symbol Connector_Generic:Conn_01x06
- removed M11: Module-vr-discrete-0.4, hellen-one-vr-discrete-0.4:vr-discrete, symbol vr-discrete-0.4:Module-vr-discrete-0.4
- removed M3: mega-mcu144-0.1, hellen-one-mega-mcu144-0.1:mega-mcu144, symbol mega-mcu144-0.1:mega-mcu144-0.1
- removed M5: Module-knock-0.2, hellen-one-knock-0.2:knock, symbol hellen-one-knock-0.2:Module-knock-0.2
- removed M6: Module-output-0.3, hellen-one-output-0.3:output, symbol hellen-one-output-0.3:Module-output-0.3
- removed M7: Module-ign8-0.2, hellen-one-ign8-0.2:ign8, symbol hellen-one-ign8-0.2:Module-ign8-0.2
- removed M8: Module-power_12and5V-0.1, hellen-one-power_12and5V-0.1:power_12and5V, symbol power_12and5V-0.1:Module-power_12and5V-0.1
- removed M9: Module-wbo-0.5, hellen-one-wbo-0.5:wbo, symbol hellen-one-wbo-0.5:Module-wbo-0.5
- removed P10, P11, P12, P13, P14, P15, P16, P17, P20, P28, P40, P41, P43, P44, P45, P46, P48, P49, P56, P61, P63, P64, P66, P67, P68, P69, P74, P80: Pad, hellen-one-common:PAD-TH, symbol hellen-one-common:Pad
- removed R10, R11, R12, R13, R2, R3, R8, R9: Jumper-Pad-Pad, hellen-one-common:PAD-0805-PAD, symbol hellen-one-common:Jumper-Pad-Pad
- removed R16, R17: 5.1k, hellen-one-common:R0603, symbol hellen-one-common:Res
- removed R20: 1.6k, hellen-one-common:R0603, symbol hellen-one-common:Res
- removed R21: 750, hellen-one-common:R0603, symbol hellen-one-common:Res
- removed R22: 10k, hellen-one-common:R0603, symbol hellen-one-common:Res
- removed R23: 0, hellen-one-common:R0603, symbol hellen-one-common:Res
- removed U1: L6205PD, hellen-one-common:SO20POWER, symbol hellen-one-common:L6205PD
- removed U3: MCP6002-xSN, Package_SO:SOIC-8_3.9x4.9mm_P1.27mm, symbol Amplifier_Operational:MCP6002-xSN
- added BT1: CR1220, kicad6-libraries:CR1220-2, symbol Device:Battery_Cell
- added D4: B5819W, hellen-one-common:SOD-123, symbol hellen-one-common:1N4148WS
- added F3, F4: 12H1500D, hellen-one-common:PAD-1206-PAD, symbol hellen-one-common:Fuse-Pad-Pad
- added H1, H2, H3, H4: M3, MountingHole:MountingHole_3.2mm_M3_Pad_Via, symbol Mechanical:MountingHole
- added J17: Conn_01x06, Connector_PinHeader_2.54mm:PinHeader_1x06_P2.54mm_Vertical, symbol Connector_Generic:Conn_01x06
- added J21: Conn_01x05_Male, Connector_Molex:Molex_SPOX_5267-05A_1x05_P2.50mm_Vertical, symbol Connector:Conn_01x05_Pin
- added J22: USB_B_Mini, hellen-one-common:USB-MINI-B-VERTICAL, symbol hellen-one-common:USB_B_Mini
- added J23: USB_C, kicad6-libraries:USB_C, symbol misc:USB_C
- added M1: Module-power_12and5V-0.3, hellen-one-power_12and5V-0.3:power_12and5V, symbol hellen-one-power_12and5V:Module-power_12and5V-0.3
- added M2: Module-knock-0.2, hellen-one-knock-0.2:knock, symbol hellen-one-knock-0.2:Module-knock-0.2
- added M3: Module-vr-discrete-0.5, hellen-one-vr-discrete-0.5:vr-discrete, symbol hellen-one-vr-discrete-0.5:Module-vr-discrete-0.5
- added M4: Module-vr-max9924-0.1, hellen-one-vr-max9924-0.1:vr-max9924, symbol vr-max9924:Module-vr-max9924-0.1
- added M5: Module-wbo-0.5, hellen-one-wbo-0.5:wbo, symbol hellen-one-wbo-0.5:Module-wbo-0.5
- added M6: Module:mega-mcu100/0.3, hellen-one-mega-mcu100-0.3:mega-mcu100, symbol hellen-one-mega-mcu100-0.3:Module{colon}mega-mcu100/0.3
- added M7: Module-can-0.1, hellen-one-can-0.1:can, symbol hellen-one-can-0.1:Module-can-0.1
- added R10, R11, R12: 10k, hellen-one-common:R0805, symbol hellen-one-common:Res
- added R13, R14: 5.6k, hellen-one-common:R0603, symbol hellen-one-common:Res
- added R2: 33k, hellen-one-common:R0603, symbol hellen-one-common:Res
- added R3: 6.8k, hellen-one-common:R0603, symbol hellen-one-common:Res
- added R6: 0, hellen-one-common:R0603, symbol hellen-one-common:Res
- added R7, R8, R9: DNP, hellen-one-common:R0805, symbol hellen-one-common:Res
- added U1: JDY-33, kicad6-libraries:JDY-33, symbol JDY-33:JDY-33
- D1, D2, D3: value 1N4148WS -> B5819W; footprint hellen-one-common:SOD-323 -> hellen-one-common:SOD-123; LCSC C2128 -> C8598
- F1: value Fuse-Pad-Pad -> 12H1500D; LCSC (none) -> C182446; MyComment DNP -> (none)
- F2: value Fuse-Pad-Pad -> 12H1500D
- P1: footprint hellen121vag:368255-2 -> 368255-2:368255-2
- R1: value 100 -> 4.7k; LCSC C22775 -> (none); MyComment (none) -> DNP
- R4: LCSC C17477 -> C17477
- R5: value 100k -> 0; LCSC C25803 -> C21189
Connections:
- net CAN+ is gone; now on net GNDA: P1.60
- net CAN- is gone; now on net GNDA: P1.58
- net IN_D1 is gone; now on net GNDA: P1.55
- net IN_D2 is gone; now on net GNDA: P1.57
- net IN_D3 is gone; now on net +5VP: P1.75
- net IN_D4 is gone; now on net +5VP: P1.76
- net IN_KNOCK1_RAW is gone; now on net +5VP: P1.106
- net IN_VSS is gone; now on net GNDA: P1.54
- net OUT_INJ5 is gone; now on net GNDA: P1.113
- net OUT_INJ8 is gone; now on net +12V: P1.24
- net OUT_VVT1_2 is gone; now on net GND: P1.115
- net V12_PERM is gone; now on net GNDA: P1.62
- net +12V: now also F2.1, P1.23, F3.1, F4.1, R2.2
- net +12V_RAW: now also D1.1 (K), D2.1 (K), D3.1 (K), G1.10, G1.15, G1.5, D4.1 (K), M1.V3 (V12_RAW); no longer C1.2, D1.2 (A), D5.1 (K), F1.2
- net +5V: now also M1.E4 (V5), M6.N22 (VCC)
- net +5VA: now also G1.14, G1.4, G1.9, M2.E1 (V5A), M3.E4 (V5_IN), M4.E4 (V5_IN), M5.W1 (V5_IN), M6.E1 (V5A_SWITCHABLE), M6.W2 (V5A_SWITCHABLE), M7.V1 (V5), R7.2, R8.2, R9.2
- net +5VP: now also P1.107, P1.71, P1.74, P1.77, P1.78, P1.79, P1.80, R1.1, M1.V4 (5VP); no longer P1.53, P1.83, P1.98
- net GND: now also G1.1, G1.11, G1.12, G1.2, G1.6, G1.7, P1.114, P1.3, BT1.2 (-), J17.3 (Pin_3), J21.4 (Pin_4), J21.5 (Pin_5), J22.5 (GND), J22.6 (Shield), J23.A1 (GND), J23.A12 (GND), J23.B1 (GND), J23.B12 (GND), J23.S1 (SHIELD), M1.S1 (GND), M2.E2 (GND), M3.G (GND), M4.G (GND), M5.E6 (LSU_H-), M5.G (GND), M6.G (GND), M7.E1 (GND), R13.1, R14.1, R3.1, U1.13 (GND); no longer P1.1, P1.2, P1.32, P1.59
- net GNDA: now also P1.52, P1.53, P1.56, P1.59, P1.61, P1.64, P1.66, P1.68, P1.98, M6.S2 (IN_D3_(PE14)), M6.S3 (IN_D2_(PE13)), M6.S4 (IN_D1_(PE12)), M6.S9 (IN_AUX1_(PB0)), M6.W1 (GNDA), R10.1, R11.1, R12.1; no longer P1.108, P1.27, P1.33, P1.36, P1.50, P1.91
- net IGN1: now also M6.W10 (IGN1_(PC13))
- net IGN2: now also M6.W9 (IGN2_(PE5))
- net IGN3: now also M6.W8 (IGN3_(PE4))
- net IGN4: now also M6.W7 (IGN4_(PE3))
- net IGN5: now also M6.W6 (IGN5_(PE2))
- net IGN6: now also M6.W5 (IGN6_(PB8))
- net INJ1: now also M6.E17 (OUT_INJ1_(PD3))
- net INJ2: now also M6.E16 (OUT_INJ2_(PA9))
- net INJ3: now also M6.E15 (OUT_INJ3_(PD11))
- net INJ4: now also M6.E14 (OUT_INJ4_(PD10))
- net INJ5: now also M6.E13 (OUT_INJ5_(PD2))
- net INJ6: now also M6.E12 (OUT_INJ6_(PA8))
- net IN_VIGN: now also F1.2, M1.V2 (IN_VIGN); no longer D3.1 (K)
- net VBAT: now also D5.1 (K), M1.E1 (VBAT), M6.N17 (VBAT)
- net VBUS: now also J21.1 (Pin_1), J22.1 (VBUS), J23.A4 (VBUS), J23.A9 (VBUS), J23.B4 (VBUS), J23.B9 (VBUS), M6.N1 (VBUS)
- net VIGN: now also M1.E3 (VIGN), M6.E5 (IN_VIGN_(PA5))
- net PIN10: now reaches P1.10
- net PIN100: now reaches P1.100
- net PIN109: now reaches P1.109
- net PIN11: now reaches P1.11
- net PIN12: now reaches P1.12
- net PIN13: now reaches P1.13
- net PIN15: now reaches P1.15
- net PIN15: now also D2.2 (A)
- net PIN16: now reaches P1.16
- net PIN16: now also D3.2 (A)
- net PIN17: now reaches P1.17
- net PIN17: now also M3.W2 (VR+)
- net PIN20: now reaches P1.20
- net PIN20: now also R1.2, M4.W1 (VR-)
- net PIN21: now reaches P1.21
- net PIN25: now reaches P1.25
- net PIN28: now reaches P1.28
- net PIN30: now reaches P1.30
- net PIN31: now reaches P1.31
- net at R4.1: now also M1.E6 (PG_5VP); no longer P1.37
- net PIN40: now reaches P1.40
- net PIN40: now also M6.S11 (IN_O2S_/_CAN_WAKEUP_(PA0))
- net PIN41: now reaches P1.41
- net PIN41: now also M6.S10 (IN_O2S2_(PA1))
- net PIN42: now reaches P1.42
- net PIN42: now also M6.S17 (IN_VSS_(PE11))
- net PIN43: now reaches P1.43
- net PIN44: now reaches P1.44
- net PIN45: now reaches P1.45
- net PIN46: now reaches P1.46
- net PIN48: now reaches P1.48
- net PIN49: now reaches P1.49
- net PIN51: now reaches P1.51
- net PIN6: now reaches P1.6
- net PIN63: now reaches P1.63
- net PIN63: now also M6.S20 (IN_IAT_(PC3))
- net PIN67: now reaches P1.67
- net PIN69: now reaches P1.69
- net PIN70: now reaches P1.70
- net at P9.1 (Pin_1): now also M7.S2 (CANH); no longer P1.9
- net +12V_PERM: now reaches P1.116
- net +12V_PERM: now also M1.V1 (V12_PERM)
- net PIN119: now reaches P1.119
- net PIN121: now reaches P1.121
- net PIN121: now also M5.E5 (LSU_H+); no longer F2.1
- net PIN108: now reaches F1.1
- net PIN108: now also P1.108; no longer P1.3
- net PIN4: now reaches P1.4
- net at D5.2 (A): now also BT1.1 (+)
- net at P7.1 (Pin_1): now also M6.N13 (UART2_TX_(PD5)), U1.2 (RXD)
- net +3.3VA: now reaches G1.13, G1.3, G1.8
- net +3.3VA: now also C1.2, M6.N15 (V33_SWITCHABLE), M7.V2 (CAN_VIO), U1.12 (3V3)
- net ADC3: now reaches R5.2
- net ADC3: now also M6.S15 (IN_KNOCK_(PA2)), R6.2
- net at P8.1 (Pin_1): now also M7.S1 (CANL)
- net at P6.1 (Pin_1): now also M6.N14 (UART2_RX_(PD6)), U1.1 (TXD)
- net +ETB_OUT renamed PIN117
- net -ETB_OUT renamed PIN118
- net ETB_EN renamed IN_KNOCK
- net IN_KNOCK: now also M2.E3 (OUT_KNOCK)
- net IN_A1 renamed VR_DISCRETE
- net VR_DISCRETE: now also M3.E3 (OUT), M6.N18 (UART8_RX_(PE0))
- net IN_A2: no longer names the net of P4.1 (Pin_1)
- net IN_A2: now also M6.N14a (LED_GREEN)
- net IN_A3: no longer names the net of P5.1 (Pin_1)
- net IN_A3: now also M6.N14b (LED_YELLOW)
- net IN_A4 renamed VR_MAX9924
- net VR_MAX9924: now also M4.E3 (OUT), M6.N19 (UART8_TX_(PE1))
- net IN_AFR renamed PIN14
- net PIN14: now also D1.2 (A)
- net IN_CAM1 renamed PIN86
- net IN_CAM2 renamed PIN87
- net IN_CLT renamed PIN93
- net IN_CRANK+ renamed PIN82
- net PIN82: now also M5.W4 (CANH), M6.W11 (CANH)
- net IN_CRANK- renamed PIN90
- net PIN90: now also M6.S19 (IN_PPS_(PA3))
- net IN_IAT renamed PIN26
- net PIN26: no longer P1.85
- net IN_MAF renamed PIN29
- net IN_MAP2 renamed PIN101
- net IN_PPS1 renamed PIN34
- net IN_PPS2 renamed PIN35
- net IN_RES1 renamed PIN38
- net PIN38: now also M6.S18 (IN_TPS_(PA4))
- net IN_RES2 renamed PIN39
- net IN_TPS1 renamed PIN92
- net IN_TPS2 renamed PIN84
- net PIN84: now also M6.S14 (IN_CRANK_(PB1)), R10.2, R7.1
- net LSU_HEAT- renamed PIN5
- net OUT_CHECK_ENGINE renamed PIN47
- net OUT_FUEL_CONSUM renamed PIN81
- net OUT_FUEL_PUMP_RELAY renamed PIN65
- net PIN65: now also M6.S21 (IN_CLT_(PC2))
- net OUT_IDLE renamed PIN105
- net PIN105: now also M5.E1 (LSU_Un)
- net OUT_IGN1 renamed PIN102
- net OUT_IGN2 renamed PIN7
- net OUT_IGN3 renamed PIN111
- net OUT_IGN4 renamed PIN94
- net OUT_IGN5 renamed PIN103
- net PIN103: now also M5.E3 (LSU_Ip)
- net OUT_IGN6 renamed PIN110
- net OUT_IGN7 renamed PIN8
- net OUT_IGN8 renamed PIN95
- net OUT_INJ1 renamed PIN96
- net PIN96: now also M5.E2 (LSU_Vm)
- net OUT_INJ2 renamed PIN89
- net PIN89: now also M6.S1 (IN_D4_(PE15)), R12.2, R9.1
- net OUT_INJ3 renamed PIN97
- net OUT_INJ4 renamed PIN88
- net PIN88: now also D4.2 (A)
- net OUT_INJ6 renamed PIN112
- net OUT_INJ7 renamed PIN19
- net PIN19: now also M4.W2 (VR+)
- net OUT_TACH renamed PG_5VP
- net PG_5VP: now also M6.N12 (SPI3_MOSI_(PC12))
- net OUT_VVT1_1 renamed PIN22
- net OUT_VVT2_B1 renamed PIN18
- net PIN18: now also M3.W1 (VR-)
- net OUT_VVT2_B2 renamed PIN120
- net OUT_WASTEGATE renamed PIN104
- new net: J23.A5 (CC1), R13.2
- new net: J23.B5 (CC2), R14.2
- new net: M6.E7 (SPI2_SCK_/_CAN2_TX_(PB13)), M7.V5 (CAN_TX)
- new net: M6.E6 (SPI2_CS_/_CAN2_RX_(PB12)), M7.V6 (CAN_RX)
- new net: J17.1 (Pin_1), M5.W8 (V33_OUT)
- new net: J17.2 (Pin_2), M5.W7 (SWCLK)
- new net: J17.4 (Pin_4), M5.W6 (SWDIO)
- new net: J17.5 (Pin_5), M5.W5 (nReset)
- new net: M5.J1 (SEL1), M5.J_GND1 (PULL_DOWN1)
- new net +3.3V: M6.N21 (V33)
- new net 5_WBO_Rtrim: M5.E4 (LSU_Rtrim)
- new net DC Driver 1/PWR: F3.2
- new net DC Driver 2/PWR: F4.2
- new net DC1_DIR: M6.E21 (OUT_PWM4_(PC8))
- new net DC1_DIS: M6.E8 (SPI2_MISO_(PB14))
- new net DC1_PWM: M6.E20 (OUT_PWM3_(PC7))
- new net DC2_DIR: M6.E9 (SPI2_MOSI_(PB15))
- new net DC2_DIS: M6.N4 (USBID_(PA10))
- new net DC2_PWM: M6.E22 (OUT_PWM5_(PC9))
- new net EGT/SPI_CS: M6.N9 (SPI3_CS_(PA15))
- new net INTERNAL_MAP: M6.S12 (IN_MAP2_(PC1))
- new net IN_AUX3: M6.S7 (IN_AUX3_(PA7))
- new net IN_KNOCK_RAW: M2.W1 (IN_KNOCK)
- new net IN_VMAIN: M6.S6 (IN_AUX4_(PC5)), R2.1, R3.2
- new net LS1: M6.E11 (OUT_INJ7_(PD15))
- new net LS2: M6.E10 (OUT_INJ8_(PD12))
- new net LS3: M6.E18 (OUT_PWM1_(PD13))
- new net LS4: M6.E19 (OUT_PWM2_(PC6))
- new net LS_HOT1: M6.W4 (IGN7_(PB9))
- new net LS_HOT2: M6.W3 (IGN8_(PE6))
- new net MISO3: M6.N11 (SPI3_MISO_(PC11))
- new net PIN1: P1.1
- new net PIN2: P1.2
- new net PIN27: P1.27
- new net PIN32: P1.32
- new net PIN33: P1.33
- new net PIN36: P1.36
- new net PIN37: M6.S13 (IN_MAP1_(PC0)), P1.37
- new net PIN50: P1.50
- new net PIN83: M5.W3 (CANL), M6.W12 (CANL), P1.83
- new net PIN85: M6.S16 (IN_CAM_(PA6)), P1.85, R11.2, R8.1
- new net PIN9: P1.9
- new net PIN91: M6.S8 (IN_AUX2_(PC4/PE9)), P1.91
- new net PWR_EN: M1.E5 (EN_5VP), M6.N20 (OUT_PWR_EN_(PE10))
- new net SCK3: M6.N10 (SPI3_SCK_(PC10))
- new net USB+: J21.3 (Pin_3), J22.3 (D+), J23.A6 (D+), J23.B6 (D+), M6.N3 (USBP_(PA12))
- new net USB-: J21.2 (Pin_2), J22.2 (D-), J23.A7 (D-), J23.B7 (D-), M6.N2 (USBM_(PA11))
- new net VREF1: M2.W2 (VREF), M6.S22 (VREF1)
- new net VR_DISCRETE_A: M3.E2 (OUT_A), R6.1
- new net VR_DISCRETE_THR: M3.E1 (Thresh_IN), M6.E23 (OUT_PWM6_(PD14))
- no-connect marks 70 -> 30
Other:
- added sheet DC Driver 1 (DC_MOTOR_0.1.kicad_sch)
- added sheet DC Driver 2 (DC_MOTOR_0.1.kicad_sch)
- added sheet EGT (egt.kicad_sch)
- added sheet Ignition (IGN6.kicad_sch)
- added sheet Injector (INJ6.kicad_sch)
- added sheet LS (LS4.kicad_sch)
- added sheet LS HOT (LS_HOT.kicad_sch)
- added sheet MAP (MAP.kicad_sch)
- note added: "#0"
- note added: "3.5A MAX Always hot capable"
- note added: "3.5A MAX Solenoid load capable"
- note added: "4"
- note added: "Bluetooth Module"
- note added: "Configurable "BUTTON" pulls"
- note added: "D"
- note added: "DC Motor"
- note added: "Flyback diodes"
- note added: "Install a 4.7 kOhm R1 resistor for using VR2- as a hall sensor input"
- note added: "LS & HS outputs"
- note added: "Move the resistor from position R143 to R145 to enable the CAN WAKEUP function. The AUX1 analog input will be unavailable."
- note added: "Move the resistor from position R6 to R5 to use ADC3 for receiving the analog signal VR-DISCRETE instead of the knock signal"
- note added: "Pin 8 may be used for shielding VR signals"
- note added: "Pin Name Recommended function B8 OUT_LS_HOT2 Fan Relay B9 OUT_LS_HOT1 Main Relay B16 OUT_LS4 Fuel Pump Replay B18 OUT_LS2 Idle Air Valve C8 GND VR Shield C15 IN_AUX3 Fuel Pressure D10 IN_BUTTON2 A/C Request All inputs are 12V-tolerant"
- note removed: "#1"
- note removed: "Board info"
- note removed: "ETB driver"
- note removed: "LEDs"
- note removed: "Ouputs"
- note removed: "Power"
- note removed: "Prototype areas"
- note removed: "TODO: knock 2"
- note removed: "http://rusefi.com/s/hellen121vag"
- note removed: "to ETB driver"

Commit message: colocacion de los componentes en un 90%
Parts:
- removed BT1: CR1220, kicad6-libraries:CR1220-2, symbol Device:Battery_Cell
- removed C1: 100n, hellen-one-common:C0603, symbol hellen-one-common:Cap
- removed D5: 1N4148WS, hellen-one-common:SOD-323, symbol hellen-one-common:1N4148WS
- removed F4: 12H1500D, hellen-one-common:PAD-1206-PAD, symbol hellen-one-common:Fuse-Pad-Pad
- removed G1, G2: PROTO_AREA, hellen-one-common:PROTO_AREA, symbol hellen-one-common:PROTO_AREA
- removed H1, H2, H3, H4: M3, MountingHole:MountingHole_3.2mm_M3_Pad_Via, symbol Mechanical:MountingHole
- removed J17: Conn_01x06, Connector_PinHeader_2.54mm:PinHeader_1x06_P2.54mm_Vertical, symbol Connector_Generic:Conn_01x06
- removed J23: USB_C, kicad6-libraries:USB_C, symbol misc:USB_C
- removed P2, P3, P4, P5, P6, P7, P8, P9: Pad, hellen-one-common:PAD-TH, symbol hellen-one-common:Pad
- removed R13, R14: 5.6k, hellen-one-common:R0603, symbol hellen-one-common:Res
- removed U1: JDY-33, kicad6-libraries:JDY-33, symbol JDY-33:JDY-33
- added U10: BTS6143D, Package_TO_SOT_SMD:TO-252-4, symbol Power_Management:BTS6143D
Connections:
- net PIN120 is gone; now on net +12V: P1.120
- net PIN6: now also M6.N14 (UART2_RX_(PD6))
- net PIN7: now also M6.N13 (UART2_TX_(PD5))
- net E7INJ8CANTX: now reaches M6.E7 (SPI2_SCK_/_CAN2_TX_(PB13)), M7.V5 (CAN_TX)
- net E6INJ7CANRX: now reaches M6.E6 (SPI2_CS_/_CAN2_RX_(PB12)), M7.V6 (CAN_RX)
- new net: U10.1 (OUT), U10.5 (OUT)
- no-connect marks 30 -> 22
Other:
- removed sheet DC Driver 2
- removed sheet MAP
- sheet Injector ports: added IN7, IN8, OUT7, OUT8; removed none
- note removed: "Bluetooth Module"
- company: andreika @ rusEFI.com -> andreika @ rusEFI.comm
